File: hardware/bare_mouse/bare_mouse/bloo.kicad_pcb (KiCad board)
At the start: 2 copper layers, 103 parts, among them J1 Serial Debug Header, J10 Conn_01x06_Female, J2 SWD Header, J4 Conn_ARM_JTAG_SWD_10, J5 SWD Header, M1 M1_Conn_Alt, M2 M2_Conn_Alt, Q0 TEFT4300, Q1 TEFT4300, Q10 Q_NMOS_GSD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

Commit message: jeremiah PCB
Parts:
- moved TP2 210.0 mm to (365.2, 73.3)
- moved U3 187.9 mm to (351.1, 85.2)
- moved TP3 173.5 mm to (330.6, 73.0)
- moved TP6 168.2 mm to (326.1, 73.0)
- moved TP4 160.3 mm to (311.9, 73.2)
- moved TP1 156.6 mm to (306.1, 73.3)
- moved L1 152.0 mm to (352.7, 136.2), turned to -90 degrees
- moved R22 146.4 mm to (364.7, 143.6), turned to 180 degrees
- moved R23 146.2 mm to (364.7, 148.3)
- moved D1 144.7 mm to (349.6, 146.0)
- moved R2 143.8 mm to (344.8, 148.3), turned to 90 degrees
- moved S1 142.2 mm to (309.4, 95.9)
- moved R6 141.8 mm to (348.8, 141.9), turned to 180 degrees
- moved R4 133.8 mm to (334.9, 160.9), turned to 180 degrees
- moved C12 130.6 mm to (352.7, 129.3), turned to 90 degrees
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Routing:
- net +5V: track 0.00 -> 153.8 mm, vias 0 -> 1
- net +3V3: track 0.00 -> 146.1 mm
- net +3.3VA: track 0.00 -> 90.3 mm, vias 0 -> 1
- net BATT_NET: track 0.00 -> 56.3 mm
- net +5V_NET: track 0.00 -> 51.3 mm
- net Net-(S1-Pad3): track 0.00 -> 19.2 mm
- net VCC: track 0.00 -> 11.8 mm
- net Net-(BT1-+): track 0.00 -> 6.97 mm
- net 3V3_BYP: track 0.00 -> 6.46 mm
- net EMIT_1: track 0.00 -> 5.36 mm
- net V_METER: track 0.00 -> 4.70 mm
- net Net-(D1-K): track 0.00 -> 4.41 mm
- net Net-(J4-~{RESET}): track 0.00 -> 4.33 mm
- net Net-(D5-A): track 0.00 -> 2.52 mm
- net Net-(D6-A): track 0.00 -> 2.48 mm
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- added copper zone on B.Cu, net GND
- added copper zone on F.Cu, net GND
Other:
- board outline added: 16.7 x 3.4 mm
