File: hardware/bare_mouse/bare_mouse/bloo.kicad_pcb (KiCad board)
At the start: 2 copper layers, 94 x 99.8 mm, 101 parts, among them J1 Serial Debug Header, J10 Conn_01x06_Female, J2 SWD Header, J4 Conn_ARM_JTAG_SWD_10, J5 SWD Header, M1 M1_Conn_Alt, M2 M2_Conn_Alt, Q0 TEFT4300, Q1 TEFT4300, Q10 Q_NMOS_GSD, Q11 Q_NMOS_GSD, Q12 Q_NMOS_GSD, Q2 TEFT4300, Q3 TEFT4300, Q8 Q_NMOS_SGD, Q9 Q_NMOS_GSD, SW1 SW, SW2 SW, SW3 SW, U1 YAAJ_BluePill_SWD_Breakout, U2 L293D, U3 LM1085-5.0, U4 APE8865Y5-33-HF-3, U5 LM66100DCKR, U6 LM66100DCKR

Commit message: connections complete
Parts:
- moved R21 1.63 mm to (316.8, 172.5)
Routing:
- net EMIT_4: track 0.00 -> 43.3 mm, vias 0 -> 4
- net +3V3: track 411.8 -> 413.4 mm
- net Net-(D6-A): track 5.11 -> 5.90 mm
Changed lines of the file:
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@@
 		(fp_arc
 			(start 1.23 9.27)
-			(mid -0.277636 8.581642)
+			(mid -0.277637 8.581642)
 			(end -1 7.09)
 			(stroke
@@
 		(fp_arc
 			(start 1.23 9.27)
-			(mid -0.277636 8.581642)
+			(mid -0.277637 8.581642)
 			(end -1 7.09)
 			(stroke
@@
 		(fp_arc
 			(start 1.23 9.27)
-			(mid -0.277636 8.581642)
+			(mid -0.277637 8.581642)
 			(end -1 7.09)
 			(stroke
@@
 		(fp_arc
 			(start 1.23 9.27)
-			(mid -0.277636 8.581642)
+			(mid -0.277637 8.581642)
 			(end -1 7.09)
 			(stroke
@@
 		(tags "resistor handsolder")
 		(property "Reference" "R3"
-			(at 3.55 -0.6 360)
+			(at 3.55 -0.6 0)
 			(layer "F.SilkS")
 			(effects
@@
 		)
 		(property "Value" "1.8k"
-			(at 4.25 0.6 360)
+			(at 4.25 0.6 0)
 			(layer "F.Fab")
 			(effects
@@
 		)
 		(fp_text user "${REFERENCE}"
-			(at 0 0 360)
+			(at 0 0 0)
 			(layer "F.Fab")
 			(effects
@@
 		(fp_arc
 			(start 1.23 9.27)
-			(mid -0.277636 8.581642)
+			(mid -0.277637 8.581642)
 			(end -1 7.09)
 			(stroke
@@
 		(fp_arc
 			(start 1.23 9.27)
-			(mid -0.277636 8.581642)
+			(mid -0.277637 8.581642)
 			(end -1 7.09)
 			(stroke
@@
 		(fp_arc
 			(start 1.23 9.27)
-			(mid -0.277636 8.581642)
+			(mid -0.277637 8.581642)
 			(end -1 7.09)
 			(stroke
@@
 		(fp_arc
 			(start 1.23 9.27)
-			(mid -0.277636 8.581642)
+			(mid -0.277637 8.581642)
 			(end -1 7.09)
 			(stroke
@@
 		(tags "capacitor handsolder")
 		(property "Reference" "C17"
-			(at 4.0625 0.5 360)
+			(at 4.0625 0.5 0)
 			(layer "B.SilkS")
 			(effects
@@
 		)
 		(property "Value" "1uF"
-			(at 4.0625 -0.75 360)
+			(at 4.0625 -0.75 0)
 			(layer "B.Fab")
 			(effects
@@
 		)
 		(fp_text user "${REFERENCE}"
-			(at 0 0 360)
+			(at 0 0 0)
 			(layer "B.Fab")
 			(effects
@@
 	(footprint "Resistor_SMD:R_1206_3216Metric_Pad1.30x1.75mm_HandSolder"
 		(layer "B.Cu")
-		(at 318.3 173)
+		(at 316.75 172.5)
 		(descr "Resistor SMD 1206 (3216 Metric), square (rectangular) end terminal, IPC_7351 nominal with elongated pad for handsoldering. (Body size source: IPC-SM-782 page 72, https://www.pcb-3d.com/wordpress/wp-content/uploads/ipc-sm-782a_amendment_1_and_2.pdf), generated with kicad-footprint-generator")
 		(tags "resistor handsolder")
@@
 		(tags "resistor handsolder")
 		(property "Reference" "R11"
-			(at -3.1 0.1 360)
+			(at -3.1 0.1 0)
 			(layer "B.SilkS")
 			(effects
@@
 		(tags "resistor handsolder")
 		(property "Reference" "R24"
-			(at -3.1 -0.1 360)
+			(at -3.1 -0.1 0)
 			(layer "B.SilkS")
 			(effects
@@
 		(tags "resistor handsolder")
 		(property "Reference" "R12"
-			(at -3.1 0 360)
+			(at -3.1 0 0)
 			(layer "B.SilkS")
 			(effects
@@
 		(tags "capacitor handsolder")
 		(property "Reference" "C18"
-			(at 4.1 0.4 360)
+			(at 4.1 0.4 0)
 			(layer "B.SilkS")
 			(effects
@@
 		)
 		(property "Value" "1uF"
-			(at 4.1 -0.9 360)
+			(at 4.1 -0.9 0)
 			(layer "B.Fab")
 			(effects
@@
 		)
 		(fp_text user "${REFERENCE}"
-			(at 0 0 360)
+			(at 0 0 0)
 			(layer "B.Fab")
 			(effects
@@
 		(tags "resistor handsolder")
 		(property "Reference" "R9"
-			(at -3.1 0 360)
+			(at -3.1 0 0)
 			(layer "B.SilkS")
 			(effects
@@
 		(tags "resistor handsolder")
 		(property "Reference" "R20"
-			(at -3.05 0.11 360)
+			(at -3.05 0.11 0)
 			(layer "B.SilkS")
 			(effects
@@
 		(tags "capacitor handsolder")
 		(property "Reference" "C11"
-			(at 4.0625 0.5 360)
+			(at 4.0625 0.5 0)
 			(layer "B.SilkS")
 			(effects
@@
 		)
 		(property "Value" "10uF"
-			(at 4.5625 -0.75 360)
+			(at 4.5625 -0.75 0)
 			(layer "B.Fab")
 			(effects
@@
 		)
 		(fp_text user "${REFERENCE}"
-			(at 0 0 360)
+			(at 0 0 0)
 			(layer "B.Fab")
 			(effects
@@
 		(tags "capacitor handsolder")
 		(property "Reference" "C12"
-			(at 4 0.5 360)
+			(at 4 0.5 0)
 			(layer "B.SilkS")
 			(effects
@@
 		)
 		(property "Value" "0.1uF"
-			(at 0 -1.9 360)
+			(at 0 -1.9 0)
 			(layer "B.Fab")
 			(effects
@@
 		)
 		(fp_text user "${REFERENCE}"
-			(at 0 0 360)
+			(at 0 0 0)
 			(layer "B.Fab")
 			(effects
@@
 	)
 	(segment
+		(start 319.08665 173.28665)
+		(end 318.3 172.5)
+		(width 0.5)
+		(layer "B.Cu")
+		(net 10)
+	)
+	(segment
 		(start 324.9 166.4)
 		(end 329.75 171.25)
@@
 	)
 	(segment
+		(start 319.56335 173.28665)
+		(end 319.08665 173.28665)
+		(width 0.5)
+		(layer "B.Cu")
+		(net 10)
+	)
+	(segment
 		(start 377.13 183.871561)
 		(end 379.751561 181.25)
@@
 	)
 	(segment
-		(start 314.3 172.2)
-		(end 314.3 169.975)
+		(start 312.5 171.775)
+		(end 314.375 169.9)
 		(width 0.5)
 		(layer "F.Cu")
@@
 	)
 	(segment
-		(start 314.3 169.975)
-		(end 314.375 169.9)
+		(start 312.5 172.2)
+		(end 312.5 171.775)
 		(width 0.5)
 		(layer "F.Cu")
@@
 	)
 	(via
-		(at 314.3 172.2)
+		(at 312.5 172.2)
 		(size 0.8)
 		(drill 0.4)
@@
 	)
 	(segment
-		(start 316.75 173)
-		(end 315.1 173)
+		(start 312.8 172.5)
+		(end 315.2 172.5)
 		(width 0.5)
 		(layer "B.Cu")
@@
 	)
 	(segment
-		(start 315.1 173)
-		(end 314.3 172.2)
+		(start 312.5 172.2)
+		(end 312.8 172.5)
 		(width 0.5)
 		(layer "B.Cu")
@@
 	)
 	(segment
+		(start 361.1 138.975)
+		(end 358.425 141.65)
+		(width 0.25)
+		(layer "F.Cu")
+		(net 59)
+	)
+	(segment
+		(start 351.25 138.5)
+		(end 349 140.75)
+		(width 0.25)
+		(layer "F.Cu")
+		(net 59)
+	)
+	(segment
+		(start 361.1 137.1)
+		(end 361.1 138.975)
+		(width 0.25)
+		(layer "F.Cu")
+		(net 59)
+	)
+	(segment
+		(start 355.275 138.5)
+		(end 351.25 138.5)
+		(width 0.25)
+		(layer "F.Cu")
+		(net 59)
+	)
+	(segment
+		(start 358.425 141.65)
+		(end 355.275 138.5)
+		(width 0.25)
+		(layer "F.Cu")
+		(net 59)
+	)
+	(segment
+		(start 347.5 152.25)
+		(end 347.5 152.53)
+		(width 0.25)
+		(layer "F.Cu")
+		(net 59)
+	)
+	(segment
+		(start 343 150.25)
+		(end 347.5 150.25)
+		(width 0.25)
+		(layer "F.Cu")
+		(net 59)
+	)
+	(segment
+		(start 349 140.75)
+		(end 349 141.75)
+		(width 0.25)
+		(layer "F.Cu")
+		(net 59)
+	)
+	(segment
+		(start 347.5 152.53)
+		(end 352.62 157.65)
+		(width 0.25)
+		(layer "F.Cu")
+		(net 59)
+	)
+	(via
+		(at 347.5 150.25)
+		(size 0.8)
+		(drill 0.4)
+		(layers "F.Cu" "B.Cu")
+		(net 59)
+	)
+	(via
+		(at 349 141.75)
+		(size 0.8)
+		(drill 0.4)
+		(layers "F.Cu" "B.Cu")
+		(net 59)
+	)
+	(via
+		(at 343 150.25)
+		(size 0.8)
+		(drill 0.4)
+		(layers "F.Cu" "B.Cu")
+		(net 59)
+	)
+	(via
+		(at 347.5 152.25)
+		(size 0.8)
+		(drill 0.4)
+		(layers "F.Cu" "B.Cu")
+		(net 59)
+	)
+	(segment
+		(start 349 144.25)
+		(end 343 150.25)
+		(width 0.25)
+		(layer "B.Cu")
+		(net 59)
+	)
+	(segment
+		(start 347.5 150.25)
+		(end 347.5 152.25)
+		(width 0.25)
+		(layer "B.Cu")
+		(net 59)
+	)
+	(segment
+		(start 349 141.75)
+		(end 349 144.25)
+		(width 0.25)
+		(layer "B.Cu")
+		(net 59)
+	)
+	(segment
