File: hardware/bare_mouse/bare_mouse/bloo.kicad_sch (KiCad schematic)
At the start: 103 parts, among them J1 Serial Debug Header, J10 Conn_01x06_Female, J2 SWD Header, J4 Conn_ARM_JTAG_SWD_10, J5 SWD Header, M1 M1_Conn_Alt, M2 M2_Conn_Alt, Q0 TEFT4300, Q1 TEFT4300, Q10 Q_NMOS_GSD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

Commit message: power ORing, SWD header, and other adam sections traced
Connections:
- net SWDCLK is gone; now on net +5V_NET: J2.3 (Pin_3), J4.4 (SWDCLK/TCK), J5.3 (Pin_3), U1.42 (SWDCLK)
- net +5V: no longer U6.6 (VOUT)
- net +5V_NET: now also U6.6 (VOUT)
Other:
- moved on the sheet: U6
Changed lines of the file:
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@@
 	)
 	(junction
+		(at 327.025 167.64)
+		(diameter 0)
+		(color 0 0 0 0)
+	)
+	(junction
 		(at 154.94 90.17)
 		(diameter 0)
@@
 	)
 	(junction
+		(at 327.025 165.1)
+		(diameter 0)
+		(color 0 0 0 0)
+	)
+	(junction
 		(at 86.36 149.225)
 		(diameter 0)
@@
 	)
 	(junction
+		(at 283.845 157.48)
+		(diameter 0)
+		(color 0 0 0 0)
+	)
+	(junction
 		(at 221.615 39.37)
 		(diameter 0)
@@
 	)
 	(junction
+		(at 282.575 160.02)
+		(diameter 0)
+		(color 0 0 0 0)
+	)
+	(junction
 		(at 123.825 169.545)
 		(diameter 0)
@@
 	)
 	(junction
+		(at 319.405 165.1)
+		(diameter 0)
+		(color 0 0 0 0)
+	)
+	(junction
 		(at 104.267 110.363)
 		(diameter 0)
@@
 	)
 	(junction
+		(at 321.945 167.64)
+		(diameter 0)
+		(color 0 0 0 0)
+	)
+	(junction
 		(at 60.325 169.545)
 		(diameter 0)
@@
 	(wire
 		(pts
+			(xy 321.945 160.02) (xy 325.12 160.02)
+		)
+		(stroke
+			(width 0)
+			(type default)
+		)
+	)
+	(wire
+		(pts
 			(xy 108.839 235.966) (xy 108.839 240.411)
 		)
@@
 	(wire
 		(pts
-			(xy 319.405 157.48) (xy 325.12 157.48)
+			(xy 319.405 165.1) (xy 327.025 165.1)
 		)
 		(stroke
@@
 	(wire
 		(pts
+			(xy 321.945 167.64) (xy 282.575 167.64)
+		)
+		(stroke
+			(width 0)
+			(type default)
+		)
+	)
+	(wire
+		(pts
 			(xy 239.395 73.025) (xy 243.205 73.025)
 		)
@@
 	(wire
 		(pts
-			(xy 278.13 160.02) (xy 300.355 160.02)
+			(xy 278.13 160.02) (xy 282.575 160.02)
 		)
 		(stroke
@@
 	(wire
 		(pts
-			(xy 307.975 132.08) (xy 307.975 162.56)
+			(xy 307.975 132.08) (xy 307.975 170.18)
+		)
+		(stroke
+			(width 0)
+			(type default)
+		)
+	)
+	(wire
+		(pts
+			(xy 283.845 165.1) (xy 283.845 157.48)
 		)
 		(stroke
@@
 	(wire
 		(pts
+			(xy 327.025 165.1) (xy 367.665 165.1)
+		)
+		(stroke
+			(width 0)
+			(type default)
+		)
+	)
+	(wire
+		(pts
 			(xy 46.355 169.545) (xy 60.325 169.545)
 		)
@@
 	(wire
 		(pts
+			(xy 367.665 167.64) (xy 327.025 167.64)
+		)
+		(stroke
+			(width 0)
+			(type default)
+		)
+	)
+	(wire
+		(pts
 			(xy 316.865 81.28) (xy 316.865 88.9)
 		)
@@
 		)
 	)
+	(wire
+		(pts
+			(xy 283.845 157.48) (xy 288.29 157.48)
+		)
+		(stroke
+			(width 0)
+			(type default)
+		)
+	)
 	(polyline
 		(pts
@@
 	(wire
 		(pts
-			(xy 307.975 162.56) (xy 325.12 162.56)
+			(xy 307.975 170.18) (xy 367.665 170.18)
 		)
 		(stroke
@@
 	(wire
 		(pts
+			(xy 327.025 167.64) (xy 321.945 167.64)
+		)
+		(stroke
+			(width 0)
+			(type default)
+		)
+	)
+	(wire
+		(pts
 			(xy 71.12 66.04) (xy 112.3068 66.04)
 		)
@@
 	(wire
 		(pts
+			(xy 282.575 160.02) (xy 300.355 160.02)
+		)
+		(stroke
+			(width 0)
+			(type default)
+		)
+	)
+	(wire
+		(pts
 			(xy 132.08 169.545) (xy 132.08 165.1)
 		)
@@
 	(wire
 		(pts
+			(xy 319.405 165.1) (xy 283.845 165.1)
+		)
+		(stroke
+			(width 0)
+			(type default)
+		)
+	)
+	(wire
+		(pts
 			(xy 352.425 92.075) (xy 339.09 92.075)
 		)
@@
 	(wire
 		(pts
+			(xy 321.945 167.64) (xy 321.945 160.02)
+		)
+		(stroke
+			(width 0)
+			(type default)
+		)
+	)
+	(wire
+		(pts
 			(xy 107.315 182.88) (xy 107.315 177.165)
 		)
@@
 	(wire
 		(pts
-			(xy 278.13 157.48) (xy 288.29 157.48)
+			(xy 278.13 157.48) (xy 283.845 157.48)
 		)
 		(stroke
@@
 	(wire
 		(pts
+			(xy 282.575 167.64) (xy 282.575 160.02)
+		)
+		(stroke
+			(width 0)
+			(type default)
+		)
+	)
+	(wire
+		(pts
 			(xy 71.12 60.96) (xy 71.12 66.04)
 		)
@@
 	(wire
 		(pts
-			(xy 319.405 137.16) (xy 319.405 157.48)
+			(xy 319.405 137.16) (xy 319.405 165.1)
 		)
 		(stroke
@@
 	(symbol
 		(lib_id "DCK6_TEX:LM66100DCKR")
-		(at 325.12 157.48 0)
+		(at 367.665 165.1 0)
+		(mirror y)
 		(unit 1)
 		(exclude_from_sim no)
@@
 		(on_board yes)
 		(dnp no)
-		(fields_autoplaced yes)
 		(property "Reference" "U6"
-			(at 345.44 147.32 0)
+			(at 347.345 154.94 0)
 			(effects
 				(font
@@
 		)
 		(property "Value" "LM66100DCKR"
-			(at 345.44 149.86 0)
+			(at 347.345 157.48 0)
 			(effects
 				(font
@@
 		)
 		(property "Footprint" "DCK6_TEX"
-			(at 325.12 157.48 0)
+			(at 367.665 165.1 0)
 			(effects
 				(font
@@
 		)
 		(property "Datasheet" "LM66100DCKR"
-			(at 325.12 157.48 0)
+			(at 367.665 165.1 0)
 			(effects
 				(font
@@
 		)
 		(property "Description" ""
-			(at 325.12 157.48 0)
+			(at 367.665 165.1 0)
 			(effects
 				(font
